Commit message: Imported upstream version '1.3.1' of 'upstream'

File: uwsim/data/scenes/g500ARM5.urdf (robot description, URDF)
Before this commit: robot girona500, 8 links, 7 joints
Links:
- link base_link: mass None -> 95
Joints:
- joint part4_to_part4_jaw2: mimic joint=part4_to_part4_jaw1 multiplier=1 offset=0 -> joint=JawOpening multiplier=1 offset=0
